Commit message: Update rotary_inverted_pendulum.urdf.xacro

File: rotary_pendulum_gz/urdf/rotary_inverted_pendulum.urdf.xacro (robot description, xacro)
@@ -7,14 +7,15 @@
   <xacro:property name="pole_initial_deg" value="3.0"/>
   <xacro:property name="pole_initial_rad" value="0.0523598776"/>
+  <link name="world"/>
   <link name="base_link">
     <inertial>
-      <origin xyz="0 0 0.05" rpy="0 0 0"/>
-      <mass value="1.0"/>
-      <inertia ixx="0.0025" ixy="0.0" ixz="0.0" iyy="0.0025" iyz="0.0" izz="0.00125"/>
+      <origin xyz="0 0 0.6" rpy="0 0 0"/>
+      <mass value="3.0"/>
+      <inertia ixx="0.360675" ixy="0.0" ixz="0.0" iyy="0.360675" iyz="0.0" izz="0.00135"/>
     </inertial>
     <visual>
-      <origin xyz="0 0 0.05" rpy="0 0 0"/>
+      <origin xyz="0 0 0.6" rpy="0 0 0"/>
       <geometry>
-        <cylinder radius="0.03" length="0.1"/>
+        <cylinder radius="0.03" length="1.2"/>
       </geometry>
       <material name="base_gray">
@@ -23,10 +24,15 @@
     </visual>
     <collision>
-      <origin xyz="0 0 0.05" rpy="0 0 0"/>
+      <origin xyz="0 0 0.6" rpy="0 0 0"/>
       <geometry>
-        <cylinder radius="0.03" length="0.1"/>
+        <cylinder radius="0.03" length="1.2"/>
       </geometry>
     </collision>
   </link>
+  <joint name="world_to_base" type="fixed">
+    <parent link="world"/>
+    <child link="base_link"/>
+    <origin xyz="0 0 0" rpy="0 0 0"/>
+  </joint>
   <link name="arm_link">
     <inertial>
@@ -76,5 +82,5 @@
     <parent link="base_link"/>
     <child link="arm_link"/>
-    <origin xyz="0 0 0.1" rpy="0 0 0"/>
+    <origin xyz="0 0 1.2" rpy="0 0 0"/>
     <axis xyz="0 0 1"/>
     <limit lower="-6.283185307" upper="6.283185307" effort="10.0" velocity="20.0"/>

Commit message: Update rotary_inverted_pendulum.urdf.xacro

File: rotary_pendulum_gz/urdf/rotary_inverted_pendulum.urdf.xacro (robot description, xacro)
@@ -91,5 +91,5 @@
     <child link="pole_link"/>
     <origin xyz="0.5 0 0" rpy="0 ${pole_initial_rad} 0"/>
-    <axis xyz="0 1 0"/>
+    <axis xyz="0 -1 0"/>
     <limit lower="-3.14159265359" upper="3.14159265359" effort="10.0" velocity="20.0"/>
     <dynamics damping="0.002" friction="0.0"/>

Commit message: Update rotary_inverted_pendulum.urdf.xacro

File: rotary_pendulum_gz/urdf/rotary_inverted_pendulum.urdf.xacro (robot description, xacro)
@@ -90,6 +90,6 @@
     <parent link="arm_link"/>
     <child link="pole_link"/>
-    <origin xyz="0.5 0 0" rpy="0 ${pole_initial_rad} 0"/>
-    <axis xyz="0 -1 0"/>
+    <origin xyz="0.5 0 0" rpy="${pole_initial_rad} 0 0"/>
+    <axis xyz="-1 0 0"/>
     <limit lower="-3.14159265359" upper="3.14159265359" effort="10.0" velocity="20.0"/>
     <dynamics damping="0.002" friction="0.0"/>

Commit message: fix

File: rotary_pendulum_gz/urdf/rotary_inverted_pendulum.urdf.xacro (robot description, xacro)
@@ -84,6 +84,6 @@
     <origin xyz="0 0 1.2" rpy="0 0 0"/>
     <axis xyz="0 0 1"/>
-    <limit lower="-6.283185307" upper="6.283185307" effort="10.0" velocity="20.0"/>
-    <dynamics damping="0.02" friction="0.0"/>
+    <limit lower="-6.283185307" upper="6.283185307" effort="30.0" velocity="30.0"/>
+    <dynamics damping="0.005" friction="0.0"/>
   </joint>
   <joint name="pole_joint" type="revolute">

Commit message: swing up

File: rotary_pendulum_gz/urdf/rotary_inverted_pendulum.urdf.xacro (robot description, xacro)
@@ -5,6 +5,6 @@
   <xacro:property name="pole_length" value="1.0"/>
   <xacro:property name="rod_radius" value="0.005"/>
-  <xacro:property name="pole_initial_deg" value="3.0"/>
-  <xacro:property name="pole_initial_rad" value="0.0523598776"/>
+  <xacro:property name="pole_initial_deg" value="-180.0"/>
+  <xacro:property name="pole_initial_rad" value="-3.14159265359"/>
   <link name="world"/>
   <link name="base_link">

Commit message: Update rotary_inverted_pendulum.urdf.xacro

File: rotary_pendulum_gz/urdf/rotary_inverted_pendulum.urdf.xacro (robot description, xacro)
@@ -2,7 +2,9 @@
 <robot name="rotary_inverted_pendulum" xmlns:xacro="http://www.ros.org/wiki/xacro">
   <xacro:arg name="controllers_file" default=""/>
-  <xacro:property name="arm_length" value="0.5"/>
+  <xacro:property name="arm_length" value="0.6"/>
   <xacro:property name="pole_length" value="1.0"/>
   <xacro:property name="rod_radius" value="0.005"/>
+  <xacro:property name="tip_mass" value="0.2"/>
+  <xacro:property name="tip_radius" value="0.03"/>
   <xacro:property name="pole_initial_deg" value="-180.0"/>
   <xacro:property name="pole_initial_rad" value="-3.14159265359"/>
@@ -37,10 +39,10 @@
   <link name="arm_link">
     <inertial>
-      <origin xyz="0.25 0 0" rpy="0 0 0"/>
+      <origin xyz="0.3 0 0" rpy="0 0 0"/>
       <mass value="0.2"/>
-      <inertia ixx="0.00000417" ixy="0.0" ixz="0.0" iyy="0.00416708" iyz="0.0" izz="0.00416708"/>
+      <inertia ixx="0.00000250" ixy="0.0" ixz="0.0" iyy="0.00600125" iyz="0.0" izz="0.00600125"/>
     </inertial>
     <visual>
-      <origin xyz="0.25 0 0" rpy="0 1.57079632679 0"/>
+      <origin xyz="0.3 0 0" rpy="0 1.57079632679 0"/>
       <geometry>
         <cylinder radius="${rod_radius}" length="${arm_length}"/>
@@ -51,5 +53,5 @@
     </visual>
     <collision>
-      <origin xyz="0.25 0 0" rpy="0 1.57079632679 0"/>
+      <origin xyz="0.3 0 0" rpy="0 1.57079632679 0"/>
       <geometry>
         <cylinder radius="${rod_radius}" length="${arm_length}"/>
@@ -90,8 +92,41 @@
     <parent link="arm_link"/>
     <child link="pole_link"/>
-    <origin xyz="0.5 0 0" rpy="${pole_initial_rad} 0 0"/>
+    <origin xyz="${arm_length} 0 0" rpy="${pole_initial_rad} 0 0"/>
     <axis xyz="-1 0 0"/>
     <limit lower="-3.14159265359" upper="3.14159265359" effort="10.0" velocity="20.0"/>
     <dynamics damping="0.002" friction="0.0"/>
+  </joint>
+  <link name="pole_tip_mass_link">
+    <inertial>
+      <origin xyz="0 0 0" rpy="0 0 0"/>
+      <mass value="${tip_mass}"/>
+      <inertia
+        ixx="${0.4 * tip_mass * tip_radius * tip_radius}"
+        ixy="0.0"
+        ixz="0.0"
+        iyy="${0.4 * tip_mass * tip_radius * tip_radius}"
+        iyz="0.0"
+        izz="${0.4 * tip_mass * tip_radius * tip_radius}"/>
+    </inertial>
+    <visual>
+      <origin xyz="0 0 0" rpy="0 0 0"/>
+      <geometry>
+        <sphere radius="${tip_radius}"/>
+      </geometry>
+      <material name="tip_mass_black">
+        <color rgba="0.05 0.05 0.05 1.0"/>
+      </material>
+    </visual>
+    <collision>
+      <origin xyz="0 0 0" rpy="0 0 0"/>
+      <geometry>
+        <sphere radius="${tip_radius}"/>
+      </geometry>
+    </collision>
+  </link>
+  <joint name="pole_tip_mass_joint" type="fixed">
+    <parent link="pole_link"/>
+    <child link="pole_tip_mass_link"/>
+    <origin xyz="0 0 ${pole_length}" rpy="0 0 0"/>
   </joint>
   <ros2_control name="GazeboSimSystem" type="system">
